Commit message: Modified pupper_test

File: robots/descriptions/pupperv2_description/urdf/pupper_test.urdf.xacro (robot description, xacro)
@@ -11,5 +11,5 @@
         <origin xyz="0 0 0" rpy="0 0 0"/>
         <geometry>
-          <mesh filename="file:///home/andrewzheng1011/champ_ws/src/terrain_champ/robots/descriptions/pupperv2_description/meshes/Hip_L.obj" scale = "1.0 1.0 1.0"/>
+          <mesh filename="file:///home/andrewzheng1011/champ_ws/src/terrain_champ/robots/descriptions/pupperv2_description/meshes_2/Hip_L.obj" scale = "1.0 1.0 1.0"/>
         </geometry>
         <material name="PupperMaterial"/>
