Commit message: Working pupperv2 model with sensors
Currently working model for all procedures... Current performance with slam is poor. May be due to poor gait resulting in noisy base and noisy imu data. Need to fix this

File: robots/descriptions/pupperv2_description/urdf/pupperv2_description.urdf (robot description, URDF)
Before this commit: robot pupperv2_description, 18 links, 17 joints
Links:
- added link camera_depth_frame
- added link camera_depth_optical_frame
- added link camera_link, mass 0.200; collision mesh filename=package://hector_sensors_description/meshes/asus_camera/asu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; visual mesh filename=package://hector_sensors_description/meshes/asus_camera/asu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
- added link camera_rgb_frame
- added link camera_rgb_optical_frame
- added link hokuyo_frame, mass 0.270; collision box size=0.058 0.058 0.087; visual mesh filename=package://hector_sensors_description/meshes/hokuyo_utm30lx/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
- added link imu_link, mass 0.001
Joints:
- added joint camera_depth_joint: type fixed, parent camera_link, child camera_depth_frame, origin xyz=0.0 0.049 0.0 rpy=0 0 0
- added joint camera_depth_optical_joint: type fixed, parent camera_depth_frame, child camera_depth_optical_frame, origin xyz=0 0 0 rpy=-1.57079632679 0.0 -1.57079632679
- added joint camera_joint: type fixed, parent base_link, child camera_link, origin xyz=0.13641 0.0 -0.05661 rpy=0 0 0
- added joint camera_rgb_joint: type fixed, parent camera_link, child camera_rgb_frame, origin xyz=0.0 0.022 0.0 rpy=0 0 0
- added joint camera_rgb_optical_joint: type fixed, parent camera_rgb_frame, child camera_rgb_optical_frame, origin xyz=0 0 0 rpy=-1.57079632679 0.0 -1.57079632679
- added joint hokuyo_joint: type fixed, parent base_link, child hokuyo_frame, origin xyz=0.0 0.0 0.08661 rpy=0 0 0
- added joint imu_joint: type fixed, parent base_link, child imu_link

File: robots/descriptions/pupperv2_description/urdf/pupperv2_description.urdf.xacro (robot description, xacro)
@@ -7,4 +7,5 @@
    <xacro:include filename="$(find pupperv2_description)/urdf/transmission.xacro"/>
    <xacro:include filename="$(find pupperv2_description)/urdf/friction.xacro"/>
+   <xacro:include filename="$(find pupperv2_description)/urdf/accessories.xacro"/>
    <!-- Enable Gazebo ROS Control -->
    <gazebo>
@@ -14,6 +15,21 @@
      </plugin>
    </gazebo>
-   <!-- Solidworks to URDF (Mostly) -->
-    <link name="base_link">
+  <!-- Accessories-->
+  <xacro:accessories base_name="base_link" base_length="${0.13641*2}"
+                    base_height="${0.04661*2}"/>
+  <gazebo>
+    <plugin name="p3d_base_controller" filename="libgazebo_ros_p3d.so">
+        <alwaysOn>true</alwaysOn>
+        <updateRate>10.0</updateRate>
+        <bodyName>base_link</bodyName>
+        <topicName>odom/ground_truth</topicName>
+        <gaussianNoise>0.01</gaussianNoise>
+        <frameName>world</frameName>
+        <xyzOffsets>0 0 0</xyzOffsets>
+        <rpyOffsets>0 0 0</rpyOffsets>
+    </plugin>
+</gazebo>
+  <!-- Solidworks to URDF (Mostly) -->
+  <link name="base_link">
     <visual>
       <origin

Commit message: Remove other robot descriptions
Remove other robot descriptions from this git repository to clean up files

File: robots/descriptions/pupperv2_description/urdf/pupperv2_description.urdf (robot description, URDF)
Before this commit: robot pupperv2_description, 25 links, 24 joints
Links:
- link FL_hip: mass 0.032035 -> 0.1082783
- link FL_lower_leg: mass 0.016718 -> 0.038000014
- link FL_toe: mass 0.0018099 -> 0.00010000005183
- link FL_upper_leg: mass 0.054665 -> 0.1419999906
- link FR_hip: mass 0.032069 -> 0.10839322
- link FR_lower_leg: mass 0.016741 -> 0.038052293
- link FR_toe: mass 0.0018099 -> 0.00010000005183
- link FR_upper_leg: mass 0.054665 -> 0.1419999906
- link RL_hip: mass 0.032035 -> 0.1082783
- link RL_lower_leg: mass 0.016718 -> 0.038000014
- link RL_toe: mass 0.0018099 -> 0.00010000005183
- link RL_upper_leg: mass 0.054665 -> 0.1419999906
- link RR_hip: mass 0.032069 -> 0.10839322
- link RR_lower_leg: mass 0.016741 -> 0.038052293
- link RR_toe: mass 0.0018099 -> 0.00010000005183
- link RR_upper_leg: mass 0.054665 -> 0.1419999906
- link base_inertia: mass 0.37691 -> 0.9839499387

File: robots/descriptions/pupperv2_description/urdf/pupperv2_description.urdf.xacro (robot description, xacro)
@@ -4,18 +4,28 @@
      For more information, please see http://wiki.ros.org/sw_urdf_exporter -->
 <robot xmlns:xacro="http://www.ros.org/wiki/xacro" name="pupperv2_description">
-   <!-- Include Files -->
-   <xacro:include filename="$(find pupperv2_description)/urdf/transmission.xacro"/>
-   <xacro:include filename="$(find pupperv2_description)/urdf/friction.xacro"/>
-   <xacro:include filename="$(find pupperv2_description)/urdf/accessories.xacro"/>
-   <!-- Enable Gazebo ROS Control -->
-   <gazebo>
-     <plugin name="gazebo_ros_control" filename="libgazebo_ros_control.so">
-       <legacyModeNS>true</legacyModeNS>
-       <robotSimType>gazebo_ros_control/DefaultRobotHWSim</robotSimType>
-     </plugin>
-   </gazebo>
+  <!-- Include Files -->
+  <xacro:include filename="$(find pupperv2_description)/urdf/transmission.xacro"/>
+  <xacro:include filename="$(find pupperv2_description)/urdf/friction.xacro"/>
+  <xacro:include filename="$(find pupperv2_description)/urdf/accessories.xacro"/>
+  <!-- Scaling Inertia Parameters from Solidworks-->
+  <xacro:property name="hip_scale" value="3.38"/>
+  <xacro:property name="lower_leg_scale" value="2.273"/>
+  <xacro:property name="toe_scale" value="5.52517E-02"/>
+  <xacro:property name="upper_leg_scale" value="2.59764"/>
+  <xacro:property name="base_scale" value="2.61057"/>
+  <!-- Enable Gazebo ROS Control -->
+  <gazebo>
+    <plugin name="gazebo_ros_control" filename="libgazebo_ros_control.so">
+      <legacyModeNS>true</legacyModeNS>
+      <robotSimType>gazebo_ros_control/DefaultRobotHWSim</robotSimType>
+    </plugin>
+  </gazebo>
+  <!-- Enable Accessories Parameter-->
+  <xacro:arg name="accessories_enabled" default="$(optenv ACCESSORIES_ENABLED 1)"/>
   <!-- Accessories-->
-  <xacro:accessories base_name="base_link" base_length="${0.13641*2}"
-                    base_height="${0.04661*2}"/>
+  <xacro:if value="$(arg accessories_enabled)">
+    <xacro:accessories base_name="base_link" base_length="${0.13641*2}"
+                        base_height="${0.04661*2}"/>
+  </xacro:if>
   <gazebo>
     <plugin name="p3d_base_controller" filename="libgazebo_ros_p3d.so">
@@ -29,5 +39,5 @@
         <rpyOffsets>0 0 0</rpyOffsets>
     </plugin>
-</gazebo>
+  </gazebo>
   <!-- Solidworks to URDF (Mostly) -->
   <link name="base_link">
@@ -61,13 +71,12 @@
           xyz="4.4516E-07 -2.0991E-07 3.7751E-06"
           rpy="0 0 0" />
-        <mass
-          value="0.37691" />
+        <mass value="${0.37691*base_scale}" />
         <inertia
-          ixx="0.00038775"
-          ixy="1.1873E-06"
-          ixz="-9.237E-07"
-          iyy="0.00085802"
-          iyz="1.7272E-07"
-          izz="0.0010086" />
+          ixx="${0.00038775*base_scale}"
+          ixy="${1.1873E-06*base_scale}"
+          ixz="${-9.237E-07*base_scale}"
+          iyy="${0.00085802*base_scale}"
+          iyz="${1.7272E-07*base_scale}"
+          izz="${0.0010086*base_scale}" />
       </inertial>
   </link>
@@ -83,12 +92,12 @@
         rpy="0 0 0" />
       <mass
-        value="0.032035" />
-      <inertia
-        ixx="5.9933E-06"
-        ixy="4.4808E-07"
-        ixz="2.4371E-10"
-        iyy="2.9538E-06"
-        iyz="6.1996E-08"
-        izz="5.7278E-06" />
+        value="${0.032035*hip_scale}" />
+      <inertia
+        ixx="${5.9933E-06*hip_scale}"
+        ixy="${4.4808E-07*hip_scale}"
+        ixz="${2.4371E-10*hip_scale}"
+        iyy="${2.9538E-06*hip_scale}"
+        iyz="${6.1996E-08*hip_scale}"
+        izz="${5.7278E-06*hip_scale}" />
     </inertial>
     <visual>
@@ -141,12 +150,12 @@
         rpy="0 0 0" />
       <mass
-        value="0.054665" />
-      <inertia
-        ixx="2.4386E-05"
-        ixy="1.682E-10"
-        ixz="2.6061E-07"
-        iyy="2.3437E-05"
-        iyz="2.7137E-07"
-        izz="6.6679E-06" />
+        value="${0.054665*upper_leg_scale}" />
+      <inertia
+        ixx="${2.4386E-05*upper_leg_scale}"
+        ixy="${1.682E-10*upper_leg_scale}"
+        ixz="${2.6061E-07*upper_leg_scale}"
+        iyy="${2.3437E-05*upper_leg_scale}"
+        iyz="${2.7137E-07*upper_leg_scale}"
+        izz="${6.6679E-06*upper_leg_scale}" />
     </inertial>
     <visual>
@@ -199,12 +208,12 @@
         rpy="0 0 0" />
       <mass
-        value="0.016718" />
-      <inertia
-        ixx="1.8319E-05"
-        ixy="-1.9835E-08"
-        ixz="2.3453E-07"
-        iyy="1.8546E-05"
-        iyz="6.7626E-07"
-        izz="5.5282E-07" />
+        value="${0.016718*lower_leg_scale}" />
+      <inertia
+        ixx="${1.8319E-05*lower_leg_scale}"
+        ixy="${-1.9835E-08*lower_leg_scale}"
+        ixz="${2.3453E-07*lower_leg_scale}"
+        iyy="${1.8546E-05*lower_leg_scale}"
+        iyz="${6.7626E-07*lower_leg_scale}"
+        izz="${5.5282E-07*lower_leg_scale}" />
     </inertial>
     <visual>
@@ -257,12 +266,12 @@
         rpy="0 0 0" />
       <mass
-        value="0.0018099" />
-      <inertia
-        ixx="5.2131E-08"
-        ixy="-1.9882E-24"
-        ixz="1.137E-08"
-        iyy="4.259E-08"
-        iyz="-9.4483E-25"
-        izz="5.6141E-08" />
+        value="${0.0018099*toe_scale}" />
+      <inertia
+        ixx="${5.2131E-08*toe_scale}"
+        ixy="${-1.9882E-24*toe_scale}"
+        ixz="${1.137E-08*toe_scale}"
+        iyy="${4.259E-08*toe_scale}"
+        iyz="${-9.4483E-25*toe_scale}"
+        izz="${5.6141E-08*toe_scale}" />
     </inertial>
     <visual>
@@ -310,12 +319,12 @@
         rpy="0 0 0" />
       <mass
-        value="0.032035" />
-      <inertia
-        ixx="5.9933E-06"
-        ixy="4.4808E-07"
-        ixz="2.4371E-10"
-        iyy="2.9538E-06"
-        iyz="6.1996E-08"
-        izz="5.7278E-06" />
+        value="${0.032035*hip_scale}" />
+      <inertia
+        ixx="${5.9933E-06*hip_scale}"
+        ixy="${4.4808E-07*hip_scale}"
+        ixz="${2.4371E-10*hip_scale}"
+        iyy="${2.9538E-06*hip_scale}"
+        iyz="${6.1996E-08*hip_scale}"
+        izz="${5.7278E-06*hip_scale}" />
     </inertial>
     <visual>
@@ -368,12 +377,12 @@
         rpy="0 0 0" />
       <mass
-        value="0.054665" />
-      <inertia
-        ixx="2.4386E-05"
-        ixy="1.682E-10"
-        ixz="2.6061E-07"
-        iyy="2.3437E-05"
-        iyz="2.7137E-07"
-        izz="6.6679E-06" />
+        value="${0.054665*upper_leg_scale}" />
+      <inertia
+        ixx="${2.4386E-05*upper_leg_scale}"
+        ixy="${1.682E-10*upper_leg_scale}"
+        ixz="${2.6061E-07*upper_leg_scale}"
+        iyy="${2.3437E-05*upper_leg_scale}"
+        iyz="${2.7137E-07*upper_leg_scale}"
+        izz="${6.6679E-06*upper_leg_scale}" />
     </inertial>
     <visual>
@@ -426,12 +435,12 @@
         rpy="0 0 0" />
       <mass
-        value="0.016718" />
-      <inertia
-        ixx="1.8319E-05"
-        ixy="-1.9835E-08"
-        ixz="2.3453E-07"
-        iyy="1.8546E-05"
-        iyz="6.7626E-07"
-        izz="5.5282E-07" />
+        value="${0.016718*lower_leg_scale}" />
+      <inertia
+        ixx="${1.8319E-05*lower_leg_scale}"
+        ixy="${-1.9835E-08*lower_leg_scale}"
+        ixz="${2.3453E-07*lower_leg_scale}"
+        iyy="${1.8546E-05*lower_leg_scale}"
+        iyz="${6.7626E-07*lower_leg_scale}"
+        izz="${5.5282E-07*lower_leg_scale}" />
     </inertial>
     <visual>
@@ -484,12 +493,12 @@
         rpy="0 0 0" />
       <mass
-        value="0.0018099" />
-      <inertia
-        ixx="5.2131E-08"
-        ixy="-1.082E-24"
-        ixz="1.137E-08"
-        iyy="4.259E-08"
-        iyz="-9.2836E-25"
-        izz="5.6141E-08" />
+        value="${0.0018099*toe_scale}" />
+      <inertia
+        ixx="${5.2131E-08*toe_scale}"
+        ixy="${-1.082E-24*toe_scale}"
+        ixz="${1.137E-08*toe_scale}"
+        iyy="${4.259E-08*toe_scale}"
+        iyz="${-9.2836E-25*toe_scale}"
+        izz="${5.6141E-08*toe_scale}" />
     </inertial>
     <visual>
@@ -537,12 +546,12 @@
         rpy="0 0 0" />
       <mass
-        value="0.032069" />
-      <inertia
-        ixx="5.9912E-06"
-        ixy="-4.4714E-07"
-        ixz="1.8534E-10"
-        iyy="2.954E-06"
-        iyz="-6.2909E-08"
-        izz="5.7295E-06" />
+        value="${0.032069*hip_scale}" />
+      <inertia
+        ixx="${5.9912E-06*hip_scale}"
+        ixy="${-4.4714E-07*hip_scale}"
+        ixz="${1.8534E-10*hip_scale}"
+        iyy="${2.954E-06*hip_scale}"
+        iyz="${-6.2909E-08*hip_scale}"
+        izz="${5.7295E-06*hip_scale}" />
     </inertial>
     <visual>
@@ -595,12 +604,12 @@
         rpy="0 0 0" />
       <mass
-        value="0.054665" />
-      <inertia
-        ixx="2.4386E-05"
-        ixy="1.682E-10"
-        ixz="-2.6061E-07"
-        iyy="2.3437E-05"
-        iyz="-2.7137E-07"
-        izz="6.6679E-06" />
+        value="${0.054665*upper_leg_scale}" />
+      <inertia
+        ixx="${2.4386E-05*upper_leg_scale}"
+        ixy="${1.682E-10*upper_leg_scale}"
+        ixz="${-2.6061E-07*upper_leg_scale}"
+        iyy="${2.3437E-05*upper_leg_scale}"
+        iyz="${-2.7137E-07*upper_leg_scale}"
+        izz="${6.6679E-06*upper_leg_scale}" />
     </inertial>
     <visual>
@@ -653,12 +662,12 @@
         rpy="0 0 0" />
       <mass
-        value="0.016741" />
-      <inertia
-        ixx="1.8313E-05"
-        ixy="1.9858E-08"
-        ixz="2.3431E-07"
-        iyy="1.854E-05"
-        iyz="-6.769E-07"
-        izz="5.5333E-07" />
+        value="${0.016741*lower_leg_scale}" />
+      <inertia
+        ixx="${1.8313E-05*lower_leg_scale}"
+        ixy="${1.9858E-08*lower_leg_scale}"
+        ixz="${2.3431E-07*lower_leg_scale}"
+        iyy="${1.854E-05*lower_leg_scale}"
+        iyz="${-6.769E-07*lower_leg_scale}"
+        izz="${5.5333E-07*lower_leg_scale}" />
     </inertial>
     <visual>
@@ -711,12 +720,12 @@
         rpy="0 0 0" />
       <mass
-        value="0.0018099" />
-      <inertia
-        ixx="5.2131E-08"
-        ixy="6.2047E-25"
-        ixz="1.137E-08"
-        iyy="4.259E-08"
-        iyz="9.8352E-25"
-        izz="5.6141E-08" />
+        value="${0.0018099*toe_scale}" />
+      <inertia
+        ixx="${5.2131E-08*toe_scale}"
+        ixy="${6.2047E-25*toe_scale}"
+        ixz="${1.137E-08*toe_scale}"
+        iyy="${4.259E-08*toe_scale}"
+        iyz="${9.8352E-25*toe_scale}"
+        izz="${5.6141E-08*toe_scale}" />
     </inertial>
     <visual>
@@ -764,12 +773,12 @@
         rpy="0 0 0" />
       <mass
-        value="0.032069" />
-      <inertia
-        ixx="5.9912E-06"
-        ixy="-4.4714E-07"
-        ixz="1.8534E-10"
-        iyy="2.954E-06"
-        iyz="-6.2909E-08"
-        izz="5.7295E-06" />
+        value="${0.032069*hip_scale}" />
+      <inertia
+        ixx="${5.9912E-06*hip_scale}"
+        ixy="${-4.4714E-07*hip_scale}"
+        ixz="${1.8534E-10*hip_scale}"
+        iyy="${2.954E-06*hip_scale}"
+        iyz="${-6.2909E-08*hip_scale}"
+        izz="${5.7295E-06*hip_scale}" />
     </inertial>
     <visual>
@@ -822,12 +831,12 @@
         rpy="0 0 0" />
       <mass
-        value="0.054665" />
-      <inertia
-        ixx="2.4386E-05"
-        ixy="1.682E-10"
-        ixz="-2.6061E-07"
-        iyy="2.3437E-05"
-        iyz="-2.7137E-07"
-        izz="6.6679E-06" />
+        value="${0.054665*upper_leg_scale}" />
+      <inertia
+        ixx="${2.4386E-05*upper_leg_scale}"
+        ixy="${1.682E-10*upper_leg_scale}"
+        ixz="${-2.6061E-07*upper_leg_scale}"
+        iyy="${2.3437E-05*upper_leg_scale}"
+        iyz="${-2.7137E-07*upper_leg_scale}"
+        izz="${6.6679E-06*upper_leg_scale}" />
     </inertial>
     <visual>
@@ -880,12 +889,12 @@
         rpy="0 0 0" />
       <mass
-        value="0.016741" />
-      <inertia
-        ixx="1.8313E-05"
-        ixy="1.9858E-08"
-        ixz="2.3431E-07"
-        iyy="1.854E-05"
-        iyz="-6.769E-07"
-        izz="5.5333E-07" />
+        value="${0.016741*lower_leg_scale}" />
+      <inertia
+        ixx="${1.8313E-05*lower_leg_scale}"
+        ixy="${1.9858E-08*lower_leg_scale}"
+        ixz="${2.3431E-07*lower_leg_scale}"
+        iyy="${1.854E-05*lower_leg_scale}"
+        iyz="${-6.769E-07*lower_leg_scale}"
+        izz="${5.5333E-07*lower_leg_scale}" />
     </inertial>
     <visual>
@@ -938,12 +947,12 @@
         rpy="0 0 0" />
       <mass
-        value="0.0018099" />
-      <inertia
-        ixx="5.2131E-08"
-        ixy="6.6018E-25"
-        ixz="1.137E-08"
-        iyy="4.259E-08"
-        iyz="2.4451E-24"
-        izz="5.6141E-08" />
+        value="${0.0018099*toe_scale}" />
+      <inertia
+        ixx="${5.2131E-08*toe_scale}"
+        ixy="${6.6018E-25*toe_scale}"
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
Commit message: Update pupperv2 to display HD model

File: robots/descriptions/pupperv2_description/urdf/pupperv2_description.urdf (robot description, URDF)
Before this commit: robot pupperv2_description, 25 links, 24 joints
Links:
- link base_link: geometry collision mesh filename=package://pupperv2_description/obj_meshes/Cube003.obj; visual mesh filename=package://pupperv2_description/obj_meshes/Body_Assembly_v3.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
- link camera_link: mass 0.200 -> 0.02
- link hokuyo_frame: mass 0.270 -> 0.027

File: robots/descriptions/pupperv2_description/urdf/pupperv2_description.urdf.xacro (robot description, xacro)
@@ -48,5 +48,5 @@
       <geometry>
         <mesh
-          filename="package://pupperv2_description/obj_meshes/Cube003.obj" />
+          filename="package://pupperv2_description/obj_meshes/Body_Assembly_v3.obj" />
       </geometry>
       <material

Commit message: Changed visual to non-simplified model

File: robots/descriptions/pupperv2_description/urdf/pupperv2_description.urdf (robot description, URDF)
Before this commit: robot pupperv2_description, 25 links, 24 joints
Links:
- link base_link: geometry collision mesh filename=package://pupperv2_description/obj_meshes/Body_Assembly_v3.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; visual mesh filename=package://pupperv2_description/obj_meshes/Body_Assembly_v3.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
